Commit message: Deleted unnecessary directories and files.
Added config/robotiq140_gripper_controller.yaml for controlling with gazebo.

Modified urdf files to make them work with gazebo simulation.
    - Added inertial tag to inner finger pads.

Added a new xacro file for plugins:
    - roboticsgroup_gazebo_mimic_joint_plugin
    - gazebo_grasp_fix

File: robotiq_2f_140_gripper_visualization/urdf/robotiq_arg2f_140_model_macro.xacro (robot description, xacro)
@@ -125,4 +125,15 @@
   <xacro:macro name="inner_finger_pad" params="prefix fingerprefix">
     <link name="${prefix}${fingerprefix}_inner_finger_pad">
+      <inertial>
+        <origin xyz="0.000299999999999317 0.0160078233491243 -0.0136945669206257" rpy="0 0 0" />
+        <mass value="0.1" />
+        <inertia
+            ixx="2.71909453810972E-06"
+            ixy="1.35402465472579E-21"
+            ixz="-7.1817349065269E-22"
+            iyy="7.69100314106116E-07"
+            iyz="6.74715432769696E-07"
+            izz="2.30315190420171E-06" />
+      </inertial>
       <visual>
         <origin xyz="0 0 0" rpy="0 0 0" />

File: robotiq_2f_140_gripper_visualization/urdf/robotiq_arg2f_transmission.xacro (robot description, xacro)
@@ -5,5 +5,5 @@
       <type>transmission_interface/SimpleTransmission</type>
       <joint name="${prefix}finger_joint">
-        <hardwareInterface>PositionJointInterface</hardwareInterface>
+        <hardwareInterface>hardware_interface/PositionJointInterface</hardwareInterface>
       </joint>
       <actuator name="${prefix}finger_joint_motor">
